File: kicad/MHzDisplayBlaster.kicad_pcb (KiCad board)
At the start: 2 copper layers, 39.6 x 31.2 mm, 6 parts, among them J1 Conn_02x15 DigitRHS, J2 Conn_02x15 DigitLHS, J3 Conn_01x02, J4 Conn_01x07, U1 DC56-11GWA

Commit message: Rev.0.2: Fixes polarity issue, improves printed info
Parts:
- removed J3: Conn_01x02, Connector_PinHeader_2.54mm:PinHeader_1x02_P2.54mm_Vertical
Connections:
- net +5V renamed Net-(J4-Pad1)
- J2 pad 2: DP1 -> DP
- J2 pad 30: DP1 -> DP
- J4 pad 2: 3 -> DIG1_CC
- J4 pad 6: DIG1_CC -> 2
- J4 pad 7: 2 -> DIG1_CC
- R1 pad 1: DIG1_CC -> 3
- U1 pad 4: DP1 -> DP
- U1 pad 9: DP2 -> DP
Routing:
- net DP: track 0.00 -> 77.4 mm, vias 0 -> 3
- net DP1: track 75.4 -> 0.00 mm, vias 2 -> 0
- net DIG1_CC: track 13.2 -> 27.9 mm, vias 0 -> 1
- net DP2: track 10.6 -> 0.00 mm
- net DIG1_D: track 40.9 -> 36.1 mm
- net 1: track 91.2 -> 87.1 mm, vias 2 -> 1
- net DIG2_C: track 32.8 -> 28.7 mm
- net 3: track 85.0 -> 87.6 mm, vias 1 -> 6
- net DIG1_C: track 35.1 -> 32.7 mm
- net 2: track 92.0 -> 90.1 mm
- net DIG2_D: track 27.0 -> 26.0 mm
Other:
- board text added: "(based on)"
- board text added: "5V"
- board text added: "Scrap Computing"
- board text added: "rev.0.2"
- board text removed: "Connect DP1-DP2"
- board text removed: "DP1"
- board text removed: "Digit 1:"
- board text removed: "Digit 2:"
- board text removed: "based on"
- board text removed: "rev.0.1"
